Commit message: hola

File: s_description/urdf/sbot.urdf.xacro (robot description, xacro)
@@ -2,14 +2,4 @@
 <robot xmlns:xacro="http://www.ros.org/wiki/xacro"
   name="srbot">
-    <!-- Colors -->
-    <material name="black">
-        <color rgba="0.0 0.0 0.0 1.0"/>
-    </material>
-    <material name="white">
-        <color rgba="1.0 1.0 1.0 1.0"/>
-    </material>
-    <material name="orange">
-        <color rgba="${255/255} ${108/255} ${10/255} 1.0"/>
-    </material>
   <!-- Links -->
   <link name="base_footprint"/>
@@ -19,15 +9,15 @@
     <inertial>
       <origin
-        xyz="-0.0356238870540699 -4.03106731601266E-05 0.121501088820445"
-        rpy="0 0 0" />
-      <mass
-        value="0.590576967248925" />
-      <inertia
-        ixx="0.0046567534727676"
-        ixy="-3.38542710266083E-06"
-        ixz="-3.65561608583262E-05"
-        iyy="0.00284799695530918"
-        iyz="1.44504078186529E-05"
-        izz="0.00695313679415047" />
+        xyz="0.0331268533143592 -0.000432916937407213 0.053571397442181"
+        rpy="0 0 0" />
+      <mass
+        value="4.83639817381771" />
+      <inertia
+        ixx="0.038861655670592"
+        ixy="0.000529616499918743"
+        ixz="0.0010173959314691"
+        iyy="0.0228312438973577"
+        iyz="3.82831626454934E-05"
+        izz="0.0575066455054651" />
     </inertial>
     <visual>
@@ -42,5 +32,5 @@
         name="">
         <color
-          rgba="0.792156862745098 0.819607843137255 0.933333333333333 1" />
+          rgba="0.964705882352941 0.964705882352941 0.952941176470588 1" />
       </material>
     </visual>
@@ -58,5 +48,5 @@
     <parent link="base_footprint"/>
     <child link="base_link"/>
-    <origin xyz="0.0 0.0 0.007" rpy="0 0 0"/>
+    <origin xyz="0.0 0.0 -0.007" rpy="0 0 0"/>
   </joint>
   <!-- Caster Link -->
@@ -65,15 +55,15 @@
     <inertial>
       <origin
-        xyz="0 -0.0053142329433118 0"
-        rpy="0 0 0" />
-      <mass
-        value="0.00502921680620392" />
-      <inertia
-        ixx="2.27248756479945E-07"
-        ixy="4.42927350742589E-24"
+        xyz="0 1.0842021724855E-19 0"
+        rpy="0 0 0" />
+      <mass
+        value="0.012201049157502" />
+      <inertia
+        ixx="9.95396738164981E-07"
+        ixy="4.75190822077712E-39"
         ixz="0"
-        iyy="2.27248756479945E-07"
-        iyz="0"
-        izz="2.27248756479945E-07" />
+        iyy="9.95396738164981E-07"
+        iyz="3.04752357318865E-23"
+        izz="9.95396738164981E-07" />
     </inertial>
     <visual>
@@ -88,16 +78,14 @@
         name="">
         <color
-          rgba="0.792156862745098 0.819607843137255 0.933333333333333 1" />
-      </material>
-    </visual>
-    <collision>
-      <origin
-        xyz="0 0 0"
-        rpy="0 0 0" />
-      <geometry>
-        <mesh
-          filename="package://s_description/meshes/front_link.STL" />
-      </geometry>
-    </collision>
+          rgba="0.749019607843137 0.749019607843137 0.749019607843137 1" />
+      </material>
+    </visual>
+    <collision>
+      <origin xyz="0 0 0" rpy="0 0 0" />
+      <geometry>
+          <!-- Cambiar a una esfera como modelo de colisión -->
+          <sphere radius="0.014281" />
+      </geometry>
+  </collision>
   </link>
   <link
@@ -105,15 +93,15 @@
     <inertial>
       <origin
-        xyz="0 0.0053142329433118 0"
-        rpy="0 0 0" />
-      <mass
-        value="0.00502921680620392" />
-      <inertia
-        ixx="2.27248756479945E-07"
-        ixy="-4.42927350742589E-24"
-        ixz="0"
-        iyy="2.27248756479945E-07"
-        iyz="0"
-        izz="2.27248756479945E-07" />
+        xyz="1.11022302462516E-16 -6.93889390390723E-18 0"
+        rpy="0 0 0" />
+      <mass
+        value="0.012201049157502" />
+      <inertia
+        ixx="9.95396738164982E-07"
+        ixy="-1.32348898008484E-23"
+        ixz="8.66927083731437E-38"
+        iyy="9.95396738164982E-07"
+        iyz="-4.80636454845762E-23"
+        izz="9.95396738164982E-07" />
     </inertial>
     <visual>
@@ -128,23 +116,21 @@
         name="">
         <color
-          rgba="0.792156862745098 0.819607843137255 0.933333333333333 1" />
-      </material>
-    </visual>
-    <collision>
-      <origin
-        xyz="0 0 0"
-        rpy="0 0 0" />
-      <geometry>
-        <mesh
-          filename="package://s_description/meshes/back_link.STL" />
-      </geometry>
-    </collision>
+          rgba="0.749019607843137 0.749019607843137 0.749019607843137 1" />
+      </material>
+    </visual>
+    <collision>
+      <origin xyz="0 0 0" rpy="0 0 0" />
+      <geometry>
+          <!-- Cambiar a una esfera como modelo de colisión -->
+          <sphere radius="0.014281" />
+      </geometry>
+  </collision>
   </link>
   <!-- Caster joint -->
   <joint
-    name="caster_joint"
+    name="caster_front_joint"
     type="revolute">
     <origin
-      xyz="0.1163 0.00023819 -0.0074277"
+      xyz="0.126 0 0.002981"
       rpy="-1.5708 0 0" />
     <parent
@@ -153,5 +139,5 @@
       link="front_link" />
     <axis
-      xyz="1 1 0" />
+      xyz="1 1 1" />
     <limit
       lower="0"
@@ -164,6 +150,6 @@
     type="revolute">
     <origin
-      xyz="-0.13399 0.0024897 -0.0073544"
-      rpy="1.5708 0 0" />
+      xyz="-0.091903 0 0.0054852"
+      rpy="-1.5708 0.077667 0" />
     <parent
       link="base_link" />
@@ -171,5 +157,5 @@
       link="back_link" />
     <axis
-      xyz="1 1 0" />
+      xyz="1 1 1" />
     <limit
       lower="0"
@@ -183,15 +169,15 @@
     <inertial>
       <origin
-        xyz="-0.0193111246434702 -0.0125131683373471 -8.98842853076509E-05"
-        rpy="0 0 0" />
-      <mass
-        value="0.182526920714148" />
-      <inertia
-        ixx="0.000396274804867751"
-        ixy="4.58837222141318E-08"
-        ixz="4.4761660275352E-08"
-        iyy="3.59896813484765E-05"
-        iyz="5.27435714959667E-09"
-        izz="0.00040519781076824" />
+        xyz="-0.0130485733276654 0.000249057510941841 -6.02472496720186E-05"
+        rpy="0 0 0" />
+      <mass
+        value="0.0447531965749244" />
+      <inertia
+        ixx="2.72747579788412E-05"
+        ixy="2.44896216734503E-07"
+        ixz="-1.00813722652812E-09"
+        iyy="3.94436239577304E-06"
+        iyz="-2.92468588333206E-09"
+        izz="2.73596827712822E-05" />
     </inertial>
     <visual>
@@ -224,6 +210,6 @@
     type="fixed">
     <origin
-      xyz="0.17228 0.0093241 0.80525"
-      rpy="0 -0.13494 0" />
+      xyz="0.161 0 0.80167"
+      rpy="0 0 0" />
     <parent
       link="base_link" />
@@ -235,26 +221,26 @@
   <!-- Platform Link -->
   <link
-    name="platform_link">
-    <inertial>
-      <origin
-        xyz="0.00524329305342652 -0.177275972417613 -3.07780343483111E-05"
-        rpy="0 0 0" />
-      <mass
-        value="5.20398239999135" />
-      <inertia
-        ixx="0.146191138478855"
-        ixy="-0.00734378144066615"
-        ixz="-6.06196116860792E-08"
-        iyy="0.0824945087110923"
-        iyz="-8.40710972180585E-08"
-        izz="0.195280459107958" />
-    </inertial>
-    <visual>
-      <origin
-        xyz="0 0 0"
-        rpy="0 0 0" />
-      <geometry>
-        <mesh
-          filename="package://s_description/meshes/platform_link.STL" />
+    name="body_link">
+    <inertial>
+      <origin
+        xyz="0.0196490463239979 -0.00759747258083848 -2.54312289516001E-06"
+        rpy="0 0 0" />
+      <mass
+        value="5.3667835678089" />
+      <inertia
+        ixx="0.191852604126404"
+        ixy="-0.00180652023375761"
+        ixz="-5.31889404871528E-05"
+        iyy="0.101149701389595"
+        iyz="5.32146569402063E-05"
+        izz="0.16932952422593" />
+    </inertial>
+    <visual>
+      <origin
+        xyz="0 0 0"
+        rpy="0 0 0" />
+      <geometry>
+        <mesh
+          filename="package://s_description/meshes/body_link.STL" />
       </geometry>
       <material
@@ -270,21 +256,127 @@
       <geometry>
         <mesh
-          filename="package://s_description/meshes/platform_link.STL" />
+          filename="package://s_description/meshes/body_link.STL" />
       </geometry>
     </collision>
   </link>
   <joint
-    name="platform_joint"
+    name="body_joint"
     type="fixed">
     <origin
-      xyz="-0.011831 -0.00043758 0.69827"
+      xyz="-0.032907 0 0.38597"
       rpy="1.5708 0 0" />
     <parent
       link="base_link" />
     <child
-      link="platform_link" />
+      link="body_link" />
     <axis
       xyz="0 0 0" />
   </joint>
+  <link
+    name="head_link">
+    <inertial>
+      <origin
+        xyz="0.00849493948773139 0.0238193372028268 0.000292060864239385"
+        rpy="0 0 0" />
+      <mass
+        value="1.07076821324471" />
+      <inertia
+        ixx="0.00952954443079687"
+        ixy="-0.000539065696028081"
+        ixz="-2.03838854365254E-05"
+        iyy="0.0107354116844579"
+        iyz="-3.6921034585701E-06"
+        izz="0.00438988033691154" />
+    </inertial>
+    <visual>
+      <origin
+        xyz="0 0 0"
+        rpy="0 0 0" />
+      <geometry>
+        <mesh
+          filename="package://s_description/meshes/head_link.STL" />
+      </geometry>
+      <material
+        name="">
+        <color
+          rgba="0.792156862745098 0.819607843137255 0.933333333333333 1" />
+      </material>
+    </visual>
+    <collision>
+      <origin
+        xyz="0 0 0"
+        rpy="0 0 0" />
+      <geometry>
+        <mesh
+          filename="package://s_description/meshes/head_link.STL" />
+      </geometry>
+    </collision>
+  </link>
+  <joint
+    name="head_joint"
+    type="fixed">
+    <origin
+      xyz="0.085023 8.857E-05 0.77053"
+      rpy="1.5708 0 -0.012333" />
+    <parent
+      link="base_link" />
+    <child
+      link="head_link" />
+    <axis
+      xyz="0 0 0" />
+  </joint>
+  <link
+    name="screen_link">
+    <inertial>
+      <origin
+        xyz="-0.00875103860863291 -0.00179905099732303 -0.0013426830002895"
+        rpy="0 0 0" />
+      <mass
+        value="0.291835845220698" />
+      <inertia
+        ixx="0.00153477162859971"
+        ixy="0.000200454438260883"
+        ixz="-5.38305946263596E-07"
+        iyy="0.00130267458234358"
+        iyz="-7.69451434566266E-07"
+        izz="0.000469996563152285" />
+    </inertial>
+    <visual>
+      <origin
+        xyz="0 0 0"
+        rpy="0 0 0" />
+      <geometry>
+        <mesh
+          filename="package://s_description/meshes/screen_link.STL" />
+      </geometry>
+      <material
+        name="">
+        <color
+          rgba="0.749019607843137 0.749019607843137 0.749019607843137 1" />
+      </material>
+    </visual>
+    <collision>
+      <origin
+        xyz="0 0 0"
+        rpy="0 0 0" />
+      <geometry>
+        <mesh
+          filename="package://s_description/meshes/screen_link.STL" />
+      </geometry>
+    </collision>
+  </link>
+  <joint
+    name="screen_joint"
+    type="fixed">
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
Commit message: ultima carga

File: s_description/urdf/sbot.urdf.xacro (robot description, xacro)
@@ -9,15 +9,15 @@
     <inertial>
       <origin
-        xyz="0.0331268533143592 -0.000432916937407213 0.053571397442181"
-        rpy="0 0 0" />
-      <mass
-        value="4.83639817381771" />
-      <inertia
-        ixx="0.038861655670592"
-        ixy="0.000529616499918743"
-        ixz="0.0010173959314691"
-        iyy="0.0228312438973577"
-        iyz="3.82831626454934E-05"
-        izz="0.0575066455054651" />
+        xyz="0.0331268533142108 -0.000432916937371297 0.0535713974422872"
+        rpy="0 0 0" />
+      <mass
+        value="4.83639817382342" />
+      <inertia
+        ixx="0.0388616556706036"
+        ixy="0.000529616499930697"
+        ixz="0.00101739593148136"
+        iyy="0.0228312438973894"
+        iyz="3.82831626396926E-05"
+        izz="0.0575066455054964" />
     </inertial>
     <visual>
@@ -446,5 +446,5 @@
         ixx="2.0932620346428E-05"
         ixy="3.39520287514895E-38"
-        ixz="1.85730748238849E-38"
+        ixz="1.85730747534606E-38"
         iyy="2.0932620346428E-05"
         iyz="6.26429932491746E-21"
@@ -453,5 +453,5 @@
     <visual>
       <origin
-        xyz="0 0 -0.0001"
+        xyz="0 0 0"
         rpy="0 0 0" />
       <geometry>
@@ -506,5 +506,5 @@
     <visual>
       <origin
-        xyz="0 0 -0.0001"
+        xyz="0 0 0"
         rpy="0 0 0" />
       <geometry>
